Commit message: feat: organize project structure, documentation, and scripts

File: ros2_ws/src/my_gazebo_package/models/car.urdf.xacro (robot description, xacro)
@@ -1,4 +1,6 @@
 <?xml version="1.0"?>
-<robot name="simplecar">
+<robot name="simplecar" xmlns:xacro="http://www.ros.org/wiki/xacro">
+    <xacro:include filename="$(find my_gazebo_package)/models/oakd_camera.urdf.xacro" />
+    <xacro:oakd_camera parent_link="base_link" />
     <!-- Colors -->
     <material name="black">
@@ -12,11 +14,11 @@
         <visual>
             <geometry>
-                <box size="1.5 0.9 0.3"/>
+                <box size="2.5 1.5 0.5"/>
             </geometry>
             <material name="blue"/>
         </visual>
         <inertial>
-            <mass value="162"/>
-            <inertia ixx="48.6" ixy="0" ixz="0" iyy="48.6" iyz="0.0" izz="48.6"/>
+            <mass value="750"/>
+            <inertia ixx="625" ixy="0" ixz="0" iyy="625" iyz="0.0" izz="625"/>
         </inertial>
     </link>
@@ -25,19 +27,19 @@
         <visual>
             <geometry>
-                <cylinder length="0.15" radius="0.3"/>
+                <cylinder length="0.25" radius="0.5"/>
             </geometry>
-            <origin rpy="1.57075 1.57075 0"/>
+            <origin rpy="1.57075 0 0"/>
             <material name="black"/>
         </visual>
         <collision>
              <geometry>
-                <cylinder length="0.15" radius="0.3"/>
+                <cylinder length="0.25" radius="0.5"/>
             </geometry>
-            <origin rpy="1.57075 1.57075 0"/>
+            <origin rpy="1.57075 0 0"/>
         </collision>
         <inertial>
-            <origin rpy="1.57075 1.57075 0"/>
-            <mass value="8.1"/>
-            <inertia ixx="97.2" ixy="0" ixz="0" iyy="97.2" iyz="0.0" izz="48.6"/>
+            <origin rpy="1.57075 0 0"/>
+            <mass value="37.5"/>
+            <inertia ixx="1250" ixy="0" ixz="0" iyy="1250" iyz="0.0" izz="625"/>
         </inertial>
     </link>
@@ -46,5 +48,5 @@
         <child link="left_front_wheel"/>
         <axis xyz="0 1 0"/>
-        <origin xyz="0 0.6 0"/>
+        <origin xyz="0 0.875 0"/>
     </joint>
     <!-- Left Front Wheel - Hinge -->
@@ -52,13 +54,13 @@
         <visual>
             <geometry>
-                <box size="0.60 0.06 0.06"/>
+                <box size="1.0 0.1 0.1"/>
             </geometry>
-            <origin xyz="0 0.3 0 " rpy="0 0 1.57075"/>
+            <origin xyz="0 0.5 0 " rpy="0 0 1.57075"/>
             <material name="black"/>
         </visual>
         <inertial>
             <origin rpy="0 0 1.57075"/>
-            <mass value="0.27"/>
-            <inertia ixx="0.001215" ixy="0" ixz="0" iyy="0.001215" iyz="0" izz="0.001215"/>
+            <mass value="1.25"/>
+            <inertia ixx="0.015625" ixy="0" ixz="0" iyy="0.015625" iyz="0" izz="0.015625"/>
         </inertial>
     </link>
@@ -67,6 +69,6 @@
         <child link="left_hinge"/>
         <axis xyz="0 0 1"/>
-        <origin xyz="0.6 0.0 0"/>
-        <limit effort="100" lower="-1.5" upper="1.5" velocity="100"/>
+        <origin xyz="1.0 0.0 0"/>
+        <limit effort="100" lower="-0.5" upper="0.5" velocity="100"/>
     </joint>
     <!-- Right Front Wheel -->
@@ -74,19 +76,19 @@
         <visual>
             <geometry>
-                <cylinder length="0.15" radius="0.3"/>
+                <cylinder length="0.25" radius="0.5"/>
             </geometry>
-            <origin rpy="-1.57075 -1.57075 0"/>
+            <origin rpy="1.57075 0 0"/>
             <material name="black"/>
         </visual>
         <collision>
              <geometry>
-                <cylinder length="0.15" radius="0.3"/>
+                <cylinder length="0.25" radius="0.5"/>
             </geometry>
-            <origin rpy="-1.57075 -1.57075 0"/>
+            <origin rpy="1.57075 0 0"/>
         </collision>
         <inertial>
-            <origin rpy="-1.57075 -1.57075 0"/>
-            <mass value="8.1"/>
-            <inertia ixx="97.2" ixy="0" ixz="0" iyy="97.2" iyz="0.0" izz="48.6"/>
+            <origin rpy="1.57075 0 0"/>
+            <mass value="37.5"/>
+            <inertia ixx="1250" ixy="0" ixz="0" iyy="1250" iyz="0.0" izz="625"/>
         </inertial>
     </link>
@@ -95,5 +97,5 @@
         <child link="right_front_wheel"/>
         <axis xyz="0 1 0"/>
-        <origin xyz="0 -0.6 0"/>
+        <origin xyz="0 -0.875 0"/>
     </joint>
     <!-- Right Front Wheel - Hinge -->
@@ -101,13 +103,13 @@
         <visual>
             <geometry>
-                <box size="0.60 0.06 0.06"/>
+                <box size="1.0 0.1 0.1"/>
             </geometry>
-            <origin xyz="0 -0.3 0 " rpy="0 0 -1.57075"/>
+            <origin xyz="0 -0.5 0 " rpy="0 0 -1.57075"/>
             <material name="black"/>
         </visual>
         <inertial>
             <origin rpy="0 0 -1.57075"/>
-            <mass value="0.27"/>
-            <inertia ixx="0.001215" ixy="0" ixz="0" iyy="0.001215" iyz="0" izz="0.001215"/>
+            <mass value="1.25"/>
+            <inertia ixx="0.015625" ixy="0" ixz="0" iyy="0.015625" iyz="0" izz="0.015625"/>
         </inertial>
     </link>
@@ -116,6 +118,6 @@
         <child link="right_hinge"/>
         <axis xyz="0 0 1"/>
-        <origin xyz="0.6 0 0"/>
-        <limit effort="100" lower="-1.5" upper="1.5" velocity="100"/>
+        <origin xyz="1.0 0 0"/>
+        <limit effort="100" lower="-0.5" upper="0.5" velocity="100"/>
     </joint>
     <!-- Left Back Wheel -->
@@ -123,19 +125,19 @@
         <visual>
             <geometry>
-                <cylinder length="0.15" radius="0.3"/>
+                <cylinder length="0.25" radius="0.5"/>
             </geometry>
-            <origin rpy="1.57075 1.57075 0"/>
+            <origin rpy="1.57075 0 0"/>
             <material name="black"/>
         </visual>
         <collision>
              <geometry>
-                <cylinder length="0.15" radius="0.3"/>
+                <cylinder length="0.25" radius="0.5"/>
             </geometry>
-            <origin rpy="1.57075 1.57075 0"/>
+            <origin rpy="1.57075 0 0"/>
         </collision>
         <inertial>
-            <origin rpy="1.57075 1.57075 0"/>
-            <mass value="8.1"/>
-            <inertia ixx="97.2" ixy="0" ixz="0" iyy="97.2" iyz="0.0" izz="48.6"/>
+            <origin rpy="1.57075 0 0"/>
+            <mass value="37.5"/>
+            <inertia ixx="1250" ixy="0" ixz="0" iyy="1250" iyz="0.0" izz="625"/>
         </inertial>
     </link>
@@ -144,5 +146,5 @@
         <child link="left_back_wheel"/>
         <axis xyz="0 1 0"/>
-        <origin xyz="-0.6 0.525 0"/>
+        <origin xyz="-1.0 0.875 0"/>
     </joint>
     <!-- Right Back Wheel -->
@@ -150,19 +152,19 @@
         <visual>
             <geometry>
-                <cylinder length="0.15" radius="0.3"/>
+                <cylinder length="0.25" radius="0.5"/>
             </geometry>
-            <origin rpy="-1.57075 -1.57075 0"/>
+            <origin rpy="1.57075 0 0"/>
             <material name="black"/>
         </visual>
         <collision>
              <geometry>
-                <cylinder length="0.15" radius="0.3"/>
+                <cylinder length="0.25" radius="0.5"/>
             </geometry>
-            <origin rpy="-1.57075 -1.57075 0"/>
+            <origin rpy="1.57075 0 0"/>
         </collision>
         <inertial>
-            <origin rpy="-1.57075 -1.57075 0"/>
-            <mass value="8.1"/>
-            <inertia ixx="97.2" ixy="0" ixz="0" iyy="97.2" iyz="0.0" izz="48.6"/>
+            <origin rpy="1.57075 0 0"/>
+            <mass value="37.5"/>
+            <inertia ixx="1250" ixy="0" ixz="0" iyy="1250" iyz="0.0" izz="625"/>
         </inertial>
     </link>
@@ -171,5 +173,5 @@
         <child link="right_back_wheel"/>
         <axis xyz="0 1 0"/>
-        <origin xyz="-0.6 -0.525 0"/>
+        <origin xyz="-1.0 -0.875 0"/>
     </joint>
 </robot>

Commit message: feat: replace car model with Ackermann-steering version and update controls

File: ros2_ws/src/my_gazebo_package/models/car.urdf.xacro (robot description, xacro)
@@ -1,177 +1,148 @@
 <?xml version="1.0"?>
-<robot name="simplecar" xmlns:xacro="http://www.ros.org/wiki/xacro">
+<robot name="ackermann_car" xmlns:xacro="http://www.ros.org/wiki/xacro">
     <xacro:include filename="$(find my_gazebo_package)/models/oakd_camera.urdf.xacro" />
-    <xacro:oakd_camera parent_link="base_link" />
-    <!-- Colors -->
+    <xacro:oakd_camera parent_link="chassis" x="0.85" y="0" z="0.46" />
+    <material name="blue">
+        <color rgba="0.5 0.5 1.0 1"/>
+    </material>
     <material name="black">
-        <color rgba="0 0 0 1"/>
+        <color rgba="0.2 0.2 0.2 1"/>
     </material>
-    <material name="blue">
-        <color rgba="0.6 0.7 0.8 1"/>
+    <material name="white">
+        <color rgba="1 1 1 1"/>
     </material>
-    <!-- Base Frame of Car -->
-    <link name="base_link">
+    <link name="base_link"/>
+    <joint name="base_link_joint" type="fixed">
+        <parent link="base_link"/>
+        <child link="chassis"/>
+        <origin xyz="0 0 0" rpy="0 0 0"/>
+    </joint>
+    <link name="chassis">
         <visual>
+            <origin xyz="-0.151427 0 0.175" rpy="0 0 0"/>
             <geometry>
-                <box size="2.5 1.5 0.5"/>
+                <box size="2.01142 1 0.568726"/>
             </geometry>
             <material name="blue"/>
         </visual>
+        <collision>
+            <origin xyz="-0.151427 0 0.175" rpy="0 0 0"/>
+            <geometry>
+                <box size="2.01142 1 0.568726"/>
+            </geometry>
+        </collision>
         <inertial>
-            <mass value="750"/>
-            <inertia ixx="625" ixy="0" ixz="0" iyy="625" iyz="0.0" izz="625"/>
+            <origin xyz="-0.151427 0 0.175" rpy="0 0 0"/>
+            <mass value="1.14395"/>
+            <inertia ixx="0.126164" ixy="0" ixz="0" iyy="0.416519" iyz="0" izz="0.481014"/>
         </inertial>
     </link>
-    <!-- Left Front Wheel -->
-    <link name="left_front_wheel">
+    <!-- Steering Links -->
+    <link name="front_left_wheel_steering_link">
         <visual>
             <geometry>
-                <cylinder length="0.25" radius="0.5"/>
+                <cylinder length="0.1" radius="0.03"/>
             </geometry>
-            <origin rpy="1.57075 0 0"/>
-            <material name="black"/>
+            <material name="white"/>
         </visual>
-        <collision>
-             <geometry>
-                <cylinder length="0.25" radius="0.5"/>
-            </geometry>
-            <origin rpy="1.57075 0 0"/>
-        </collision>
         <inertial>
-            <origin rpy="1.57075 0 0"/>
-            <mass value="37.5"/>
-            <inertia ixx="1250" ixy="0" ixz="0" iyy="1250" iyz="0.0" izz="625"/>
+            <mass value="0.5"/>
+            <inertia ixx="0.0153" ixy="0" ixz="0" iyy="0.025" iyz="0" izz="0.0153"/>
         </inertial>
     </link>
-    <joint name="left_hinge_to_left_front_wheel" type="continuous">
-        <parent link="left_hinge"/>
-        <child link="left_front_wheel"/>
-        <axis xyz="0 1 0"/>
-        <origin xyz="0 0.875 0"/>
+    <joint name="front_left_wheel_steering_joint" type="revolute">
+        <parent link="chassis"/>
+        <child link="front_left_wheel_steering_link"/>
+        <origin xyz="0.554283 0.5 0.02" rpy="0 0 0"/>
+        <axis xyz="0 0 1"/>
+        <limit lower="-0.6" upper="0.6" velocity="1.0" effort="25"/>
     </joint>
-    <!-- Left Front Wheel - Hinge -->
-    <link name="left_hinge">
+    <link name="front_right_wheel_steering_link">
         <visual>
             <geometry>
-                <box size="1.0 0.1 0.1"/>
+                <cylinder length="0.1" radius="0.03"/>
             </geometry>
-            <origin xyz="0 0.5 0 " rpy="0 0 1.57075"/>
-            <material name="black"/>
+            <material name="white"/>
         </visual>
         <inertial>
-            <origin rpy="0 0 1.57075"/>
-            <mass value="1.25"/>
-            <inertia ixx="0.015625" ixy="0" ixz="0" iyy="0.015625" iyz="0" izz="0.015625"/>
+            <mass value="0.5"/>
+            <inertia ixx="0.0153" ixy="0" ixz="0" iyy="0.025" iyz="0" izz="0.0153"/>
         </inertial>
     </link>
-    <joint name="base_to_left_hinge" type="revolute">
-        <parent link="base_link"/>
-        <child link="left_hinge"/>
+    <joint name="front_right_wheel_steering_joint" type="revolute">
+        <parent link="chassis"/>
+        <child link="front_right_wheel_steering_link"/>
+        <origin xyz="0.554283 -0.5 0.02" rpy="0 0 0"/>
         <axis xyz="0 0 1"/>
-        <origin xyz="1.0 0.0 0"/>
-        <limit effort="100" lower="-0.5" upper="0.5" velocity="100"/>
+        <limit lower="-0.6" upper="0.6" velocity="1.0" effort="25"/>
     </joint>
-    <!-- Right Front Wheel -->
-    <link name="right_front_wheel">
-        <visual>
-            <geometry>
-                <cylinder length="0.25" radius="0.5"/>
-            </geometry>
-            <origin rpy="1.57075 0 0"/>
-            <material name="black"/>
-        </visual>
-        <collision>
-             <geometry>
-                <cylinder length="0.25" radius="0.5"/>
-            </geometry>
-            <origin rpy="1.57075 0 0"/>
-        </collision>
-        <inertial>
-            <origin rpy="1.57075 0 0"/>
-            <mass value="37.5"/>
-            <inertia ixx="1250" ixy="0" ixz="0" iyy="1250" iyz="0.0" izz="625"/>
-        </inertial>
-    </link>
-    <joint name="right_hinge_to_right_front_wheel" type="continuous">
-        <parent link="right_hinge"/>
-        <child link="right_front_wheel"/>
-        <axis xyz="0 1 0"/>
-        <origin xyz="0 -0.875 0"/>
-    </joint>
-    <!-- Right Front Wheel - Hinge -->
-    <link name="right_hinge">
-        <visual>
-            <geometry>
-                <box size="1.0 0.1 0.1"/>
-            </geometry>
-            <origin xyz="0 -0.5 0 " rpy="0 0 -1.57075"/>
-            <material name="black"/>
-        </visual>
-        <inertial>
-            <origin rpy="0 0 -1.57075"/>
-            <mass value="1.25"/>
-            <inertia ixx="0.015625" ixy="0" ixz="0" iyy="0.015625" iyz="0" izz="0.015625"/>
-        </inertial>
-    </link>
-    <joint name="base_to_right_hinge" type="revolute">
-        <parent link="base_link"/>
-        <child link="right_hinge"/>
-        <axis xyz="0 0 1"/>
-        <origin xyz="1.0 0 0"/>
-        <limit effort="100" lower="-0.5" upper="0.5" velocity="100"/>
-    </joint>
-    <!-- Left Back Wheel -->
-    <link name="left_back_wheel">
-        <visual>
-            <geometry>
-                <cylinder length="0.25" radius="0.5"/>
-            </geometry>
-            <origin rpy="1.57075 0 0"/>
-            <material name="black"/>
-        </visual>
-        <collision>
-             <geometry>
-                <cylinder length="0.25" radius="0.5"/>
-            </geometry>
-            <origin rpy="1.57075 0 0"/>
-        </collision>
-        <inertial>
-            <origin rpy="1.57075 0 0"/>
-            <mass value="37.5"/>
-            <inertia ixx="1250" ixy="0" ixz="0" iyy="1250" iyz="0.0" izz="625"/>
-        </inertial>
-    </link>
-    <joint name="base_to_left_back_wheel" type="continuous">
-        <parent link="base_link"/>
-        <child link="left_back_wheel"/>
-        <axis xyz="0 1 0"/>
-        <origin xyz="-1.0 0.875 0"/>
-    </joint>
-    <!-- Right Back Wheel -->
-    <link name="right_back_wheel">
-        <visual>
-            <geometry>
-                <cylinder length="0.25" radius="0.5"/>
-            </geometry>
-            <origin rpy="1.57075 0 0"/>
-            <material name="black"/>
-        </visual>
-        <collision>
-             <geometry>
-                <cylinder length="0.25" radius="0.5"/>
-            </geometry>
-            <origin rpy="1.57075 0 0"/>
-        </collision>
-        <inertial>
-            <origin rpy="1.57075 0 0"/>
-            <mass value="37.5"/>
-            <inertia ixx="1250" ixy="0" ixz="0" iyy="1250" iyz="0.0" izz="625"/>
-        </inertial>
-    </link>
-    <joint name="base_to_right_back_wheel" type="continuous">
-        <parent link="base_link"/>
-        <child link="right_back_wheel"/>
-        <axis xyz="0 1 0"/>
-        <origin xyz="-1.0 -0.875 0"/>
-    </joint>
+    <!-- Wheels Macro -->
+    <xacro:macro name="wheel" params="name parent_link *origin">
+        <link name="${name}">
+            <visual>
+                <origin xyz="0 0 0" rpy="1.570796 0 0"/>
+                <geometry>
+                    <cylinder length="0.15" radius="0.3"/>
+                </geometry>
+                <material name="black"/>
+            </visual>
+            <collision>
+                <origin xyz="0 0 0" rpy="1.570796 0 0"/>
+                <geometry>
+                    <cylinder length="0.15" radius="0.3"/>
+                </geometry>
+            </collision>
+            <inertial>
+                <origin xyz="0 0 0" rpy="1.570796 0 0"/>
+                <mass value="2"/>
+                <inertia ixx="0.145833" ixy="0" ixz="0" iyy="0.145833" iyz="0" izz="0.125"/>
+            </inertial>
+        </link>
+        <joint name="${name}_joint" type="continuous">
+            <parent link="${parent_link}"/>
+            <child link="${name}"/>
+            <xacro:insert_block name="origin"/>
+            <axis xyz="0 1 0"/>
+        </joint>
+    </xacro:macro>
+    <xacro:wheel name="front_left_wheel" parent_link="front_left_wheel_steering_link">
+        <origin xyz="0 0.125029 -0.045" rpy="0 0 0"/>
+    </xacro:wheel>
+    <xacro:wheel name="front_right_wheel" parent_link="front_right_wheel_steering_link">
+        <origin xyz="0 -0.125029 -0.045" rpy="0 0 0"/>
+    </xacro:wheel>
+    <xacro:wheel name="rear_left_wheel" parent_link="chassis">
+        <origin xyz="-0.957138 0.625029 -0.025" rpy="0 0 0"/>
+    </xacro:wheel>
+    <xacro:wheel name="rear_right_wheel" parent_link="chassis">
+        <origin xyz="-0.957138 -0.625029 -0.025" rpy="0 0 0"/>
+    </xacro:wheel>
+    <gazebo>
+        <plugin
+            filename="gz-sim-ackermann-steering-system"
+            name="gz::sim::systems::AckermannSteering">
+            <left_joint>front_left_wheel_joint</left_joint>
+            <left_joint>rear_left_wheel_joint</left_joint>
+            <right_joint>front_right_wheel_joint</right_joint>
+            <right_joint>rear_right_wheel_joint</right_joint>
+            <left_steering_joint>front_left_wheel_steering_joint</left_steering_joint>
+            <right_steering_joint>front_right_wheel_steering_joint</right_steering_joint>
+            <kingpin_width>1.0</kingpin_width>
+            <steering_limit>0.5</steering_limit>
+            <wheel_base>1.0</wheel_base>
+            <wheel_separation>1.25</wheel_separation>
+            <wheel_radius>0.3</wheel_radius>
+            <topic>cmd_vel</topic>
+            <odom_topic>odom</odom_topic>
+            <min_velocity>-1</min_velocity>
+            <max_velocity>1</max_velocity>
+            <min_acceleration>-3</min_acceleration>
+            <max_acceleration>3</max_acceleration>
+        </plugin>
+        <plugin
+            filename="gz-sim-joint-state-publisher-system"
+            name="gz::sim::systems::JointStatePublisher">
+            <topic>joint_states</topic>
+        </plugin>
+    </gazebo>
 </robot>

File: ros2_ws/src/my_gazebo_package/models/oakd_camera.urdf.xacro (robot description, xacro)
@@ -1,9 +1,9 @@
 <?xml version="1.0"?>
 <robot xmlns:xacro="http://www.ros.org/wiki/xacro">
-  <xacro:macro name="oakd_camera" params="parent_link">
+  <xacro:macro name="oakd_camera" params="parent_link x:=1.0 y:=0 z:=0.25">
     <joint name="camera_base_joint" type="fixed">
       <parent link="${parent_link}"/>
       <child link="camera_base_link"/>
-      <origin xyz="1.0 0 0.25" rpy="0 0 0"/>
+      <origin xyz="${x} ${y} ${z}" rpy="0 0 0"/>
     </joint>
     <link name="camera_base_link">
