Commit message: feat: implement RTAB-Map SLAM with lossless depth and OPi optimized bridge

File: ros2_ws/src/my_gazebo_package/models/car.urdf.xacro (robot description, xacro)
@@ -34,8 +34,30 @@
         <inertial>
             <origin xyz="-0.151427 0 0.175" rpy="0 0 0"/>
-            <mass value="1.14395"/>
-            <inertia ixx="0.126164" ixy="0" ixz="0" iyy="0.416519" iyz="0" izz="0.481014"/>
+            <mass value="50.0"/>
+            <inertia ixx="5.0" ixy="0" ixz="0" iyy="17.0" iyz="0" izz="20.0"/>
         </inertial>
     </link>
+    <!-- IMU Link and Sensor -->
+    <link name="imu_link">
+        <inertial>
+            <mass value="0.1"/>
+            <inertia ixx="0.0001" ixy="0" ixz="0" iyy="0.0001" iyz="0" izz="0.0001"/>
+        </inertial>
+    </link>
+    <joint name="imu_joint" type="fixed">
+        <parent link="chassis"/>
+        <child link="imu_link"/>
+        <origin xyz="0 0 0" rpy="0 0 0"/>
+    </joint>
+    <gazebo reference="imu_link">
+        <sensor name="imu_sensor" type="imu">
+            <always_on>1</always_on>
+            <update_rate>100</update_rate>
+            <visualize>true</visualize>
+            <topic>imu</topic>
+            <plugin filename="gz-sim-imu-system" name="gz::sim::systems::Imu">
+            </plugin>
+        </sensor>
+    </gazebo>
     <!-- Steering Links -->
     <link name="front_left_wheel_steering_link">
@@ -47,5 +69,5 @@
         </visual>
         <inertial>
-            <mass value="0.5"/>
+            <mass value="5.0"/>
             <inertia ixx="0.0153" ixy="0" ixz="0" iyy="0.025" iyz="0" izz="0.0153"/>
         </inertial>
@@ -56,5 +78,5 @@
         <origin xyz="0.554283 0.5 0.02" rpy="0 0 0"/>
         <axis xyz="0 0 1"/>
-        <limit lower="-0.6" upper="0.6" velocity="1.0" effort="25"/>
+        <limit lower="-0.6" upper="0.6" velocity="10.0" effort="1000"/>
     </joint>
     <link name="front_right_wheel_steering_link">
@@ -66,5 +88,5 @@
         </visual>
         <inertial>
-            <mass value="0.5"/>
+            <mass value="5.0"/>
             <inertia ixx="0.0153" ixy="0" ixz="0" iyy="0.025" iyz="0" izz="0.0153"/>
         </inertial>
@@ -75,5 +97,5 @@
         <origin xyz="0.554283 -0.5 0.02" rpy="0 0 0"/>
         <axis xyz="0 0 1"/>
-        <limit lower="-0.6" upper="0.6" velocity="1.0" effort="25"/>
+        <limit lower="-0.6" upper="0.6" velocity="10.0" effort="1000"/>
     </joint>
     <!-- Wheels Macro -->
@@ -95,6 +117,6 @@
             <inertial>
                 <origin xyz="0 0 0" rpy="1.570796 0 0"/>
-                <mass value="2"/>
-                <inertia ixx="0.145833" ixy="0" ixz="0" iyy="0.145833" iyz="0" izz="0.125"/>
+                <mass value="15.0"/>
+                <inertia ixx="0.5" ixy="0" ixz="0" iyy="0.5" iyz="0" izz="0.7"/>
             </inertial>
         </link>
@@ -104,4 +126,5 @@
             <xacro:insert_block name="origin"/>
             <axis xyz="0 1 0"/>
+            <limit effort="5000" velocity="100"/>
         </joint>
     </xacro:macro>
@@ -135,8 +158,8 @@
             <topic>cmd_vel</topic>
             <odom_topic>odom</odom_topic>
-            <min_velocity>-1</min_velocity>
-            <max_velocity>1</max_velocity>
-            <min_acceleration>-3</min_acceleration>
-            <max_acceleration>3</max_acceleration>
+            <min_velocity>-13.41</min_velocity>
+            <max_velocity>13.41</max_velocity>
+            <min_acceleration>-30</min_acceleration>
+            <max_acceleration>30</max_acceleration>
         </plugin>
         <plugin

File: ros2_ws/src/my_gazebo_package/models/oakd_camera.urdf.xacro (robot description, xacro)
@@ -36,4 +36,10 @@
       </inertial>
     </link>
+    <joint name="camera_optical_joint" type="fixed">
+      <parent link="camera_link_rgb"/>
+      <child link="camera_link_optical"/>
+      <origin xyz="0 0 0" rpy="-1.570796 0 -1.570796"/>
+    </joint>
+    <link name="camera_link_optical"/>
     <joint name="camera_left_joint" type="fixed">
       <parent link="camera_base_link"/>
@@ -72,20 +78,20 @@
     <!-- Gazebo sensor definitions -->
     <gazebo reference="camera_link_rgb">
-      <sensor type="camera" name="rgb_camera">
+      <sensor type="rgbd_camera" name="oakd_rgbd_camera">
         <update_rate>30.0</update_rate>
         <camera name="head">
           <horizontal_fov>1.396</horizontal_fov>
           <image>
-            <width>1920</width>
-            <height>1080</height>
+            <width>640</width>
+            <height>480</height>
             <format>R8G8B8</format>
           </image>
           <clip>
             <near>0.02</near>
-            <far>300</far>
+            <far>30</far>
           </clip>
         </camera>
-        <topic>/oakd/rgb/image_raw</topic>
-        <camera_info_topic>/oakd/rgb/camera_info</camera_info_topic>
+        <topic>/oakd/rgbd_camera</topic>
+        <gz_frame_id>camera_link_rgb</gz_frame_id>
       </sensor>
     </gazebo>
