Commit message: feat: implement synchronized RGB-D streaming for OAK-D on edge device
- Updated OAK-D URDF with metric depth noise profiles
- Implemented high-fidelity 16-bit PNG depth streamer
- Configured RTAB-Map for in-memory DB and optimized sync for RK3588
- Updated deployment scripts for direct Ethernet hardware connection
- Added EDGE_DEVICE.md specification and requirements

File: ros2_ws/src/my_gazebo_package/models/oakd_camera.urdf.xacro (robot description, xacro)
@@ -45,5 +45,5 @@
       <parent link="camera_base_link"/>
       <child link="camera_link_left"/>
-      <origin xyz="0 0.0375 0" rpy="0 0 0"/>
+      <origin xyz="0 0.075 0" rpy="0 0 0"/>
     </joint>
     <link name="camera_link_left">
@@ -62,5 +62,5 @@
       <parent link="camera_base_link"/>
       <child link="camera_link_right"/>
-      <origin xyz="0 -0.0375 0" rpy="0 0 0"/>
+      <origin xyz="0 -0.075 0" rpy="0 0 0"/>
     </joint>
     <link name="camera_link_right">
@@ -83,15 +83,20 @@
           <horizontal_fov>1.396</horizontal_fov>
           <image>
-            <width>640</width>
-            <height>480</height>
+            <width>1280</width>
+            <height>800</height>
             <format>R8G8B8</format>
           </image>
           <clip>
-            <near>0.02</near>
-            <far>30</far>
+            <near>0.7</near>
+            <far>30.0</far>
           </clip>
+          <noise>
+            <type>gaussian</type>
+            <mean>0.0</mean>
+            <stddev>0.007</stddev>
+          </noise>
         </camera>
         <topic>/oakd/rgbd_camera</topic>
-        <gz_frame_id>camera_link_rgb</gz_frame_id>
+        <gz_frame_id>camera_link_optical</gz_frame_id>
       </sensor>
     </gazebo>
@@ -100,5 +105,5 @@
         <update_rate>30.0</update_rate>
         <camera name="left">
-          <horizontal_fov>1.22</horizontal_fov>
+          <horizontal_fov>1.396</horizontal_fov>
           <image>
             <width>1280</width>
@@ -119,5 +124,5 @@
         <update_rate>30.0</update_rate>
         <camera name="right">
-          <horizontal_fov>1.22</horizontal_fov>
+          <horizontal_fov>1.396</horizontal_fov>
           <image>
             <width>1280</width>
