Commit message: feat: implement autonomous racing validation stack

File: server_sim/src/my_gazebo_package/models/car.urdf.xacro (robot description, xacro)
@@ -78,5 +78,5 @@
         <origin xyz="0.554283 0.5 0.02" rpy="0 0 0"/>
         <axis xyz="0 0 1"/>
-        <limit lower="-0.6" upper="0.6" velocity="10.0" effort="1000"/>
+        <limit lower="-0.6108" upper="0.6108" velocity="10.0" effort="1000"/>
     </joint>
     <link name="front_right_wheel_steering_link">
@@ -97,5 +97,5 @@
         <origin xyz="0.554283 -0.5 0.02" rpy="0 0 0"/>
         <axis xyz="0 0 1"/>
-        <limit lower="-0.6" upper="0.6" velocity="10.0" effort="1000"/>
+        <limit lower="-0.6108" upper="0.6108" velocity="10.0" effort="1000"/>
     </joint>
     <!-- Wheels Macro -->
@@ -152,6 +152,7 @@
             <right_steering_joint>front_right_wheel_steering_joint</right_steering_joint>
             <kingpin_width>1.0</kingpin_width>
-            <steering_limit>0.5</steering_limit>
-            <wheel_base>1.0</wheel_base>
+            <steering_limit>0.6108</steering_limit>
+            <steer_p_gain>3.0</steer_p_gain>
+            <wheel_base>1.511</wheel_base>
             <wheel_separation>1.25</wheel_separation>
             <wheel_radius>0.3</wheel_radius>
